File: Addressable_Driver/Addressable_Driver.kicad_pcb (KiCad board)
At the start: 2 copper layers, 50.4 x 77.8 mm, 16 parts, among them J1 Conn_Coaxial_Power, J2 Screw_Terminal_01x04, J4 Conn_01x04_Male, SW1 SW_SPST, U1 ESP32_DevKit_V1_DOIT, U2 74LS125

Commit message: Adds resistor for data output for addressable version
Parts:
- added R2: R_US, Resistor_THT:R_Axial_DIN0207_L6.3mm_D2.5mm_P7.62mm_Horizontal, F.Cu at (148.8, 97.1)
Connections:
- J2 pad 2: /D_out_shifted -> Net-(J2-Pad2)
- U2 pad 3: /D_out_shifted -> Net-(U2-Pad3)
Routing:
- net /D_out_shifted: track 47.6 -> 0.00 mm
- net Net-(U2-Pad3): track 0.00 -> 31.9 mm
- net Net-(J2-Pad2): track 0.00 -> 12.5 mm
Changed lines of the file:
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@@
   (net 19 "unconnected-(U1-Pad6)")
   (net 20 "unconnected-(U1-Pad7)")
-  (net 21 "/D_out_shifted")
+  (net 21 "Net-(J2-Pad2)")
   (net 22 "unconnected-(U1-Pad18)")
   (net 23 "unconnected-(U1-Pad19)")
@@
   (net 31 "/D_out")
   (net 32 "unconnected-(J2-Pad3)")
+  (net 33 "Net-(U2-Pad3)")
   (footprint "MountingHole:MountingHole_2.2mm_M2" (layer "F.Cu")
     (at 152.95 125.6)
@@
     (fp_circle (center 0 0) (end 2.45 0) (layer "F.CrtYd") (width 0.05) (fill none))
     (pad "" np_thru_hole circle locked (at 0 0) (size 2.2 2.2) (drill 2.2) (layers *.Cu *.Mask))
+  )
+  (footprint "Resistor_THT:R_Axial_DIN0207_L6.3mm_D2.5mm_P7.62mm_Horizontal" (layer "F.Cu")
+    (at 148.85 97.1 90)
+    (descr "Resistor, Axial_DIN0207 series, Axial, Horizontal, pin pitch=7.62mm, 0.25W = 1/4W, length*diameter=6.3*2.5mm^2, http://cdn-reichelt.de/documents/datenblatt/B400/1_4W%23YAG.pdf")
+    (tags "Resistor Axial_DIN0207 series Axial Horizontal pin pitch 7.62mm 0.25W = 1/4W length 6.3mm diameter 2.5mm")
+    (property "Sheetfile" "Addressable_Driver.kicad_sch")
+    (property "Sheetname" "")
+    (attr through_hole)
+    (fp_text reference "R2" (at 3.81 -2.37 90) (layer "F.SilkS")
+      (effects (font (size 1 1) (thickness 0.15)))
+    )
+    (fp_text value "R_US" (at 3.81 2.37 90) (layer "F.Fab")
+      (effects (font (size 1 1) (thickness 0.15)))
+    )
+    (fp_text user "${REFERENCE}" (at 3.81 0 90) (layer "F.Fab")
+      (effects (font (size 1 1) (thickness 0.15)))
+    )
+    (fp_line (start 0.54 1.04) (end 0.54 1.37) (layer "F.SilkS") (width 0.12))
+    (fp_line (start 0.54 -1.37) (end 7.08 -1.37) (layer "F.SilkS") (width 0.12))
+    (fp_line (start 0.54 1.37) (end 7.08 1.37) (layer "F.SilkS") (width 0.12))
+    (fp_line (start 0.54 -1.04) (end 0.54 -1.37) (layer "F.SilkS") (width 0.12))
+    (fp_line (start 7.08 -1.37) (end 7.08 -1.04) (layer "F.SilkS") (width 0.12))
+    (fp_line (start 7.08 1.37) (end 7.08 1.04) (layer "F.SilkS") (width 0.12))
+    (fp_line (start 8.67 1.5) (end 8.67 -1.5) (layer "F.CrtYd") (width 0.05))
+    (fp_line (start -1.05 -1.5) (end -1.05 1.5) (layer "F.CrtYd") (width 0.05))
+    (fp_line (start 8.67 -1.5) (end -1.05 -1.5) (layer "F.CrtYd") (width 0.05))
+    (fp_line (start -1.05 1.5) (end 8.67 1.5) (layer "F.CrtYd") (width 0.05))
+    (fp_line (start 6.96 1.25) (end 6.96 -1.25) (layer "F.Fab") (width 0.1))
+    (fp_line (start 0.66 1.25) (end 6.96 1.25) (layer "F.Fab") (width 0.1))
+    (fp_line (start 0.66 -1.25) (end 0.66 1.25) (layer "F.Fab") (width 0.1))
+    (fp_line (start 7.62 0) (end 6.96 0) (layer "F.Fab") (width 0.1))
+    (fp_line (start 6.96 -1.25) (end 0.66 -1.25) (layer "F.Fab") (width 0.1))
+    (fp_line (start 0 0) (end 0.66 0) (layer "F.Fab") (width 0.1))
+    (pad "1" thru_hole circle locked (at 0 0 90) (size 1.6 1.6) (drill 0.8) (layers *.Cu *.Mask)
+      (net 33 "Net-(U2-Pad3)") (pintype "passive"))
+    (pad "2" thru_hole oval locked (at 7.62 0 90) (size 1.6 1.6) (drill 0.8) (layers *.Cu *.Mask)
+      (net 21 "Net-(J2-Pad2)") (pintype "passive"))
+    (model "${KICAD6_3DMODEL_DIR}/Resistor_THT.3dshapes/R_Axial_DIN0207_L6.3mm_D2.5mm_P7.62mm_Horizontal.wrl"
+      (offset (xyz 0 0 0))
+      (scale (xyz 1 1 1))
+      (rotate (xyz 0 0 0))
+    )
   )
   (footprint "MountingHole:MountingHole_2.2mm_M2" locked (layer "F.Cu")
@@
       (net 31 "/D_out") (pintype "input"))
     (pad "3" thru_hole oval locked (at 0 5.08 270) (size 1.6 1.6) (drill 0.8) (layers *.Cu *.Mask)
-      (net 21 "/D_out_shifted") (pintype "tri_state"))
+      (net 33 "Net-(U2-Pad3)") (pintype "tri_state"))
     (pad "4" thru_hole oval locked (at 0 7.62 270) (size 1.6 1.6) (drill 0.8) (layers *.Cu *.Mask))
     (pad "5" thru_hole oval locked (at 0 10.16 270) (size 1.6 1.6) (drill 0.8) (layers *.Cu *.Mask))
@@
       (net 2 "GND") (pinfunction "Pin_1") (pintype "passive"))
     (pad "2" thru_hole circle locked (at 5.08 0 90) (size 3 3) (drill 1.52) (layers *.Cu *.Mask)
-      (net 21 "/D_out_shifted") (pinfunction "Pin_2") (pintype "passive"))
+      (net 21 "Net-(J2-Pad2)") (pinfunction "Pin_2") (pintype "passive"))
     (pad "3" thru_hole circle locked (at 10.16 0 90) (size 3 3) (drill 1.52) (layers *.Cu *.Mask)
       (net 32 "unconnected-(J2-Pad3)") (pinfunction "Pin_3") (pintype "passive+no_connect"))
@@
   (segment (start 143.5 120.89) (end 131.48 108.87) (width 0.25) (layer "F.Cu") (net 3))
   (segment (start 131.48 108.87) (end 131.25 108.87) (width 0.25) (layer "F.Cu") (net 3))
-  (segment (start 141.155789 104.904511) (end 150.35 95.7103) (width 0.25) (layer "F.Cu") (net 21))
-  (segment (start 126.17 101.25) (end 127.294511 102.374511) (width 0.25) (layer "F.Cu") (net 21))
-  (segment (start 139.855489 104.904511) (end 141.155789 104.904511) (width 0.25) (layer "F.Cu") (net 21))
-  (segment (start 150.35 95.7103) (end 150.35 80.32) (width 0.25) (layer "F.Cu") (net 21))
-  (segment (start 150.35 80.32) (end 152.25 78.42) (width 0.25) (layer "F.Cu") (net 21))
-  (segment (start 127.294511 102.374511) (end 137.325489 102.374511) (width 0.25) (layer "F.Cu") (net 21))
-  (segment (start 137.325489 102.374511) (end 139.855489 104.904511) (width 0.25) (layer "F.Cu") (net 21))
+  (segment (start 148.85 89.48) (end 148.85 81.82) (width 0.25) (layer "F.Cu") (net 21))
+  (segment (start 148.85 81.82) (end 152.25 78.42) (width 0.25) (layer "F.Cu") (net 21))
   (segment (start 140.6 111.31) (end 140.69 111.4) (width 0.25) (layer "F.Cu") (net 29))
   (segment (start 136.35 111.31) (end 140.6 111.31) (width 0.25) (layer "F.Cu") (net 29))
@@
   (segment (start 131.35 98.61) (end 136.35 98.61) (width 0.25) (layer "F.Cu") (net 31))
   (segment (start 128.71 101.25) (end 131.35 98.61) (width 0.25) (layer "F.Cu") (net 31))
+  (segment (start 148.85 97.80656) (end 148.85 97.1) (width 0.25) (layer "F.Cu") (net 33))
+  (segment (start 134.776511 109.856511) (end 136.800049 109.856511) (width 0.25) (layer "F.Cu") (net 33))
+  (segment (start 136.800049 109.856511) (end 148.85 97.80656) (width 0.25) (layer "F.Cu") (net 33))
+  (segment (start 126.17 101.25) (end 134.776511 109.856511) (width 0.25) (layer "F.Cu") (net 33))
   (zone (net 1) (net_name "+12V") (layer "B.Cu") (hatch edge 0.508)
     (connect_pads yes (clearance 0.508))

Commit message: Finishes addressable driver
Connections:
- U1 pad 19: unconnected-(U1-Pad19) -> Net-(U1-Pad19)
- U1 pad 21: /D_out -> unconnected-(U1-Pad21)
- U2 pad 2: /D_out -> Net-(U1-Pad19)
Routing:
- net /D_out: track 8.73 -> 0.00 mm
- net Net-(U1-Pad19): track 0.00 -> 8.65 mm
Changed lines of the file:
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@@
   (net 21 "Net-(J2-Pad2)")
   (net 22 "unconnected-(U1-Pad18)")
-  (net 23 "unconnected-(U1-Pad19)")
+  (net 23 "Net-(R2-Pad1)")
   (net 24 "unconnected-(U1-Pad20)")
   (net 25 "unconnected-(U1-Pad27)")
@@
   (net 29 "+3V3")
   (net 30 "/GPIO0")
-  (net 31 "/D_out")
-  (net 32 "unconnected-(J2-Pad3)")
-  (net 33 "Net-(U2-Pad3)")
+  (net 31 "unconnected-(J2-Pad3)")
+  (net 32 "unconnected-(U1-Pad21)")
+  (net 33 "Net-(U1-Pad19)")
   (footprint "MountingHole:MountingHole_2.2mm_M2" (layer "F.Cu")
     (at 152.95 125.6)
@@
     (fp_line (start 0 0) (end 0.66 0) (layer "F.Fab") (width 0.1))
     (pad "1" thru_hole circle locked (at 0 0 90) (size 1.6 1.6) (drill 0.8) (layers *.Cu *.Mask)
-      (net 33 "Net-(U2-Pad3)") (pintype "passive"))
+      (net 23 "Net-(R2-Pad1)") (pintype "passive"))
     (pad "2" thru_hole oval locked (at 7.62 0 90) (size 1.6 1.6) (drill 0.8) (layers *.Cu *.Mask)
       (net 21 "Net-(J2-Pad2)") (pintype "passive"))
@@
       (net 22 "unconnected-(U1-Pad18)") (pinfunction "IO15") (pintype "bidirectional+no_connect"))
     (pad "19" thru_hole circle locked (at 12.7 27.94) (size 1.524 1.524) (drill 0.762) (layers *.Cu *.Mask)
-      (net 23 "unconnected-(U1-Pad19)") (pinfunction "IO2") (pintype "bidirectional+no_connect"))
+      (net 33 "Net-(U1-Pad19)") (pinfunction "IO2") (pintype "bidirectional"))
     (pad "20" thru_hole circle locked (at 12.7 25.4) (size 1.524 1.524) (drill 0.762) (layers *.Cu *.Mask)
       (net 24 "unconnected-(U1-Pad20)") (pinfunction "IO4") (pintype "bidirectional+no_connect"))
     (pad "21" thru_hole circle locked (at 12.7 22.86) (size 1.524 1.524) (drill 0.762) (layers *.Cu *.Mask)
-      (net 31 "/D_out") (pinfunction "IO16") (pintype "bidirectional"))
+      (net 32 "unconnected-(U1-Pad21)") (pinfunction "IO16") (pintype "bidirectional+no_connect"))
     (pad "22" thru_hole circle locked (at 12.7 20.32) (size 1.524 1.524) (drill 0.762) (layers *.Cu *.Mask)
       (net 30 "/GPIO0") (pinfunction "IO17") (pintype "bidirectional"))
@@
       (net 2 "GND") (pintype "input"))
     (pad "2" thru_hole oval locked (at 0 2.54 270) (size 1.6 1.6) (drill 0.8) (layers *.Cu *.Mask)
-      (net 31 "/D_out") (pintype "input"))
+      (net 33 "Net-(U1-Pad19)") (pintype "input"))
     (pad "3" thru_hole oval locked (at 0 5.08 270) (size 1.6 1.6) (drill 0.8) (layers *.Cu *.Mask)
-      (net 33 "Net-(U2-Pad3)") (pintype "tri_state"))
+      (net 23 "Net-(R2-Pad1)") (pintype "tri_state"))
     (pad "4" thru_hole oval locked (at 0 7.62 270) (size 1.6 1.6) (drill 0.8) (layers *.Cu *.Mask))
     (pad "5" thru_hole oval locked (at 0 10.16 270) (size 1.6 1.6) (drill 0.8) (layers *.Cu *.Mask))
@@
       (net 21 "Net-(J2-Pad2)") (pinfunction "Pin_2") (pintype "passive"))
     (pad "3" thru_hole circle locked (at 10.16 0 90) (size 3 3) (drill 1.52) (layers *.Cu *.Mask)
-      (net 32 "unconnected-(J2-Pad3)") (pinfunction "Pin_3") (pintype "passive+no_connect"))
+      (net 31 "unconnected-(J2-Pad3)") (pinfunction "Pin_3") (pintype "passive+no_connect"))
     (pad "4" thru_hole circle locked (at 15.24 0 90) (size 3 3) (drill 1.52) (layers *.Cu *.Mask)
       (net 1 "+12V") (pinfunction "Pin_4") (pintype "passive"))
@@
   (segment (start 148.85 89.48) (end 148.85 81.82) (width 0.25) (layer "F.Cu") (net 21))
   (segment (start 148.85 81.82) (end 152.25 78.42) (width 0.25) (layer "F.Cu") (net 21))
+  (segment (start 148.85 97.80656) (end 148.85 97.1) (width 0.25) (layer "F.Cu") (net 23))
+  (segment (start 134.776511 109.856511) (end 136.800049 109.856511) (width 0.25) (layer "F.Cu") (net 23))
+  (segment (start 136.800049 109.856511) (end 148.85 97.80656) (width 0.25) (layer "F.Cu") (net 23))
+  (segment (start 126.17 101.25) (end 134.776511 109.856511) (width 0.25) (layer "F.Cu") (net 23))
   (segment (start 140.6 111.31) (end 140.69 111.4) (width 0.25) (layer "F.Cu") (net 29))
   (segment (start 136.35 111.31) (end 140.6 111.31) (width 0.25) (layer "F.Cu") (net 29))
@@
   (segment (start 140.69 103.78) (end 140.69 100.41) (width 0.25) (layer "F.Cu") (net 30))
   (segment (start 132.374511 92.094511) (end 136.35 96.07) (width 0.25) (layer "F.Cu") (net 30))
-  (segment (start 131.35 98.61) (end 136.35 98.61) (width 0.25) (layer "F.Cu") (net 31))
-  (segment (start 128.71 101.25) (end 131.35 98.61) (width 0.25) (layer "F.Cu") (net 31))
-  (segment (start 148.85 97.80656) (end 148.85 97.1) (width 0.25) (layer "F.Cu") (net 33))
-  (segment (start 134.776511 109.856511) (end 136.800049 109.856511) (width 0.25) (layer "F.Cu") (net 33))
-  (segment (start 136.800049 109.856511) (end 148.85 97.80656) (width 0.25) (layer "F.Cu") (net 33))
-  (segment (start 126.17 101.25) (end 134.776511 109.856511) (width 0.25) (layer "F.Cu") (net 33))
+  (segment (start 128.71 101.25) (end 131.15 103.69) (width 0.25) (layer "F.Cu") (net 33))
+  (segment (start 131.15 103.69) (end 136.35 103.69) (width 0.25) (layer "F.Cu") (net 33))
   (zone (net 1) (net_name "+12V") (layer "B.Cu") (hatch edge 0.508)
     (connect_pads yes (clearance 0.508))
