File: Addressable_Driver/Addressable_Driver.kicad_sch (KiCad schematic)
At the start: 8 parts, among them J1 Conn_Coaxial_Power, J2 Screw_Terminal_01x04, J4 Conn_01x04_Male, SW1 SW_SPST, U1 ESP32_DevKit_V1_DOIT, U2 74LS125

Commit message: Adds resistor for data output for addressable version
Parts:
- added R2: R_US, Resistor_THT:R_Axial_DIN0207_L6.3mm_D2.5mm_P7.62mm_Horizontal, symbol Device:R_US
Connections:
- net D_out_shifted: no longer names the net of U2.3
- net D_out_shifted: now also R2.1; no longer J2.2 (Pin_2)
- new net: J2.2 (Pin_2), R2.2
Changed lines of the file:
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@@
+    (stroke (width 0) (type default) (color 0 0 0 0))
+  )
+  (wire (pts (xy 146.05 69.85) (xy 149.86 69.85))
     (stroke (width 0) (type default) (color 0 0 0 0))
   )
@@
     (stroke (width 0) (type default) (color 0 0 0 0))
   )
-  (wire (pts (xy 134.62 69.85) (xy 149.86 69.85))
-    (stroke (width 0) (type default) (color 0 0 0 0))
-  )
   (wire (pts (xy 100.33 76.2) (xy 127 76.2))
     (stroke (width 0) (type default) (color 0 0 0 0))
@@
     (stroke (width 0) (type default) (color 0 0 0 0))
   )
+  (wire (pts (xy 134.62 69.85) (xy 138.43 69.85))
+    (stroke (width 0) (type default) (color 0 0 0 0))
+  )
   (wire (pts (xy 156.21 78.74) (xy 152.4 78.74))
     (stroke (width 0) (type default) (color 0 0 0 0))
@@
   (wire (pts (xy 100.33 76.2) (xy 100.33 82.55))
     (stroke (width 0) (type default) (color 0 0 0 0))
-  )
-  (label "D_out_shifted" (at 135.89 69.85 0)
-    (effects (font (size 1.27 1.27)) (justify left bottom))
   )
   (label "D_out" (at 107.95 69.85 0)
@@
     )
     (pin "1")
+  )
+  (symbol (lib_id "Device:R_US") (at 142.24 69.85 90) (unit 1)
+    (in_bom yes) (on_board yes) (fields_autoplaced)
+    (property "Reference" "R2" (id 0) (at 142.24 64.9945 90))
+    (property "Value" "R_US" (id 1) (at 142.24 67.7696 90))
+    (property "Footprint" "Resistor_THT:R_Axial_DIN0207_L6.3mm_D2.5mm_P7.62mm_Horizontal" (id 2) (at 142.494 68.834 90)
+      (effects (font (size 1.27 1.27)) hide)
+    )
+    (property "Datasheet" "~" (id 3) (at 142.24 69.85 0)
+      (effects (font (size 1.27 1.27)) hide)
+    )
+    (pin "1")
+    (pin "2")
   )
   (symbol (lib_id "Connector:Conn_01x04_Male") (at 119.38 113.03 180) (unit 1)
@@
       (reference "R1") (unit 1) (value "10k") (footprint "Resistor_THT:R_Axial_DIN0207_L6.3mm_D2.5mm_P7.62mm_Horizontal")
     )
+    (path "/20d98c48-32ab-46ba-bdf6-6e1aeca2df62"
+      (reference "R2") (unit 1) (value "R_US") (footprint "Resistor_THT:R_Axial_DIN0207_L6.3mm_D2.5mm_P7.62mm_Horizontal")
+    )
     (path "/b7cf2839-b1c0-4185-bd2b-8b40d3060ac9"

Commit message: Finishes addressable driver
Connections:
- net at U1.19 (IO2): now also U2.2
- net D_out: no longer names the net of U1.21 (IO16)
- net D_out: no longer U2.2
- no-connect marks 25 -> 26
Changed lines of the file:
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@@
   (no_connect (at 87.63 82.55))
   (no_connect (at 87.63 46.99))
+  (no_connect (at 88.9 46.99))
+  (no_connect (at 87.63 54.61))
   (no_connect (at 87.63 49.53))
   (no_connect (at 57.15 29.21))
@@
   (no_connect (at 87.63 62.23))
   (no_connect (at 87.63 59.69))
-  (no_connect (at 87.63 34.29))
   (no_connect (at 87.63 41.91))
   (no_connect (at 87.63 87.63))
@@
     (stroke (width 0) (type default) (color 0 0 0 0))
   )
-  (wire (pts (xy 87.63 54.61) (xy 95.25 54.61))
-    (stroke (width 0) (type default) (color 0 0 0 0))
-  )
-  (wire (pts (xy 95.25 54.61) (xy 95.25 69.85))
-    (stroke (width 0) (type default) (color 0 0 0 0))
-  )
   (wire (pts (xy 153.67 71.12) (xy 156.21 71.12))
     (stroke (width 0) (type default) (color 0 0 0 0))
@@
   )
   (wire (pts (xy 107.95 113.03) (xy 114.3 113.03))
+    (stroke (width 0) (type default) (color 0 0 0 0))
+  )
+  (wire (pts (xy 95.25 34.29) (xy 95.25 69.85))
     (stroke (width 0) (type default) (color 0 0 0 0))
   )
@@
   )
   (wire (pts (xy 72.39 20.32) (xy 72.39 19.05))
+    (stroke (width 0) (type default) (color 0 0 0 0))
+  )
+  (wire (pts (xy 95.25 34.29) (xy 87.63 34.29))
     (stroke (width 0) (type default) (color 0 0 0 0))
   )
@@
     (stroke (width 0) (type default) (color 0 0 0 0))
   )
-  (label "D_out" (at 107.95 69.85 0)
-    (effects (font (size 1.27 1.27)) (justify left bottom))
-  )
   (label "GPIO0" (at 104.14 57.15 0)
